Commit message: feat: add the control module
The control module contains the Jacobian based control of the joints
for trajectory tracking.

File: src/fret/urdf/scara.xacro (robot description, xacro)
@@ -62,4 +62,13 @@
      <!-- Dummy root link with no inertia to satisfy KDL (avoid root inertia warning) -->
      <link name="base_root"/>
+     <!-- World link: anchors the robot to the Gazebo world frame.
+          Without this fixed joint, Gazebo treats the robot as free-floating
+          and the TF tree is disconnected from the world frame. -->
+     <link name="world"/>
+     <joint name="world_to_base_root" type="fixed">
+          <parent link="world"/>
+          <child link="base_root"/>
+          <origin xyz="0 0 0" rpy="0 0 0"/>
+     </joint>
      <!-- Link 0: Base plate + pedestal cylinder -->
       <link name="base_link">

Commit message: fix: setup scara joint control

File: src/fret/urdf/scara.xacro (robot description, xacro)
@@ -576,3 +576,46 @@
           <origin xyz="0 0 0" rpy="0 0 0"/>
      </joint>
+     <!-- ============================================================ -->
+     <!-- ros2_control: velocity interfaces for Gazebo Harmonic SITL   -->
+     <!--   j1_velocity = 375*pi/180 ≈ 6.545 rad/s                    -->
+     <!--   j2_velocity = 600*pi/180 ≈ 10.472 rad/s                   -->
+     <!--   j3_velocity = 1.111 m/s                                    -->
+     <!-- ============================================================ -->
+     <ros2_control name="GazeboSystem" type="system">
+          <hardware>
+               <plugin>gz_ros2_control/GazeboSimSystem</plugin>
+          </hardware>
+          <joint name="joint_arm_0">
+               <command_interface name="velocity">
+                    <param name="min">-6.545</param>
+                    <param name="max">6.545</param>
+               </command_interface>
+               <state_interface name="position"/>
+               <state_interface name="velocity"/>
+          </joint>
+          <joint name="joint_arm_1">
+               <command_interface name="velocity">
+                    <param name="min">-10.472</param>
+                    <param name="max">10.472</param>
+               </command_interface>
+               <state_interface name="position"/>
+               <state_interface name="velocity"/>
+          </joint>
+          <joint name="joint_extension">
+               <command_interface name="velocity">
+                    <param name="min">-1.111</param>
+                    <param name="max">1.111</param>
+               </command_interface>
+               <state_interface name="position"/>
+               <state_interface name="velocity"/>
+          </joint>
+     </ros2_control>
+     <!-- Gazebo Harmonic plugin: starts the ros2_control controller manager
+          inside the simulation process and loads the controller YAML. -->
+     <gazebo>
+          <plugin filename="gz_ros2_control-system"
+                  name="gz_ros2_control::GazeboSimROS2ControlPlugin">
+               <parameters>$(find fret)/config/controllers/ros2_control.yaml</parameters>
+          </plugin>
+     </gazebo>
 </robot>
